File: ETROC_to_FPGA.kicad_pcb (KiCad board)
At the start: 4 copper layers, 100 x 100 mm, 82 parts, among them J1 TF06L-80S-0.5SH_800_, J2 TF06L-80S-0.5SH_800_, J3 ASP-134604-01, J5 Conn_Coaxial, J6 Barrel_Jack, J7 Conn_01x03, U1 PCA9306, U2 MIC69502WR, U3 504102B00000G, U4 PCA9306, U6 MIC69502WR

Commit message: Fabricated ETROC_to_FPGA_v1
Parts:
- added C19: 10n, Capacitor_SMD:C_0805_2012Metric_Pad1.18x1.45mm_HandSolder, F.Cu at (56.5, -65.5)
- added R26: 2.2k, Resistor_SMD:R_0805_2012Metric_Pad1.20x1.40mm_HandSolder, F.Cu at (39.4, -49.0)
- added R27: 2.2k, Resistor_SMD:R_0805_2012Metric_Pad1.20x1.40mm_HandSolder, F.Cu at (42.4, -49.0)
- added R53: 2.2k, Resistor_SMD:R_0805_2012Metric_Pad1.20x1.40mm_HandSolder, F.Cu at (42.8, -25.5)
- added R54: 2.2k, Resistor_SMD:R_0805_2012Metric_Pad1.20x1.40mm_HandSolder, F.Cu at (45.8, -25.5)
- added R66: 2.2k, Resistor_SMD:R_0805_2012Metric_Pad1.20x1.40mm_HandSolder, F.Cu at (46.2, -49.0)
- added R67: 2.2k, Resistor_SMD:R_0805_2012Metric_Pad1.20x1.40mm_HandSolder, F.Cu at (49.2, -49.0)
- added R75: 2.2k, Resistor_SMD:R_0805_2012Metric_Pad1.20x1.40mm_HandSolder, F.Cu at (51.7, -25.5)
- added R76: 2.2k, Resistor_SMD:R_0805_2012Metric_Pad1.20x1.40mm_HandSolder, F.Cu at (54.7, -25.5)
- C1: renamed from C10; value 10uF ? -> 10uF; footprint Capacitor_SMD:C_0603_1608Metric -> Capacitor_SMD:C_0805_2012Metric_Pad1.18x1.45mm_HandSolder
- C12: renamed from C2; footprint Capacitor_SMD:C_0603_1608Metric -> Capacitor_SMD:C_0805_2012Metric_Pad1.18x1.45mm_HandSolder
- C17: renamed from C5; value C -> 100n; footprint Capacitor_SMD:C_0201_0603Metric_Pad0.64x0.40mm_HandSolder -> Capacitor_SMD:C_0805_2012Metric_Pad1.18x1.45mm_HandSolder
- C18: renamed from C6; value C -> 100n; footprint Capacitor_SMD:C_0201_0603Metric_Pad0.64x0.40mm_HandSolder -> Capacitor_SMD:C_0805_2012Metric_Pad1.18x1.45mm_HandSolder
- C2: renamed from C3; footprint Capacitor_SMD:C_0201_0603Metric_Pad0.64x0.40mm_HandSolder -> Capacitor_SMD:C_0805_2012Metric_Pad1.18x1.45mm_HandSolder
- C20: renamed from C11; value C -> 100n; footprint Capacitor_SMD:C_0201_0603Metric_Pad0.64x0.40mm_HandSolder -> Capacitor_SMD:C_0805_2012Metric_Pad1.18x1.45mm_HandSolder
- C21: renamed from C12; value C -> 100n; footprint Capacitor_SMD:C_0201_0603Metric_Pad0.64x0.40mm_HandSolder -> Capacitor_SMD:C_0805_2012Metric_Pad1.18x1.45mm_HandSolder
- C22: renamed from C13; value C -> 100n; footprint Capacitor_SMD:C_0201_0603Metric_Pad0.64x0.40mm_HandSolder -> Capacitor_SMD:C_0805_2012Metric_Pad1.18x1.45mm_HandSolder
- C23: renamed from C14; value C -> 100n; footprint Capacitor_SMD:C_0201_0603Metric_Pad0.64x0.40mm_HandSolder -> Capacitor_SMD:C_0805_2012Metric_Pad1.18x1.45mm_HandSolder
- C3: renamed from C4; footprint Capacitor_SMD:C_0201_0603Metric_Pad0.64x0.40mm_HandSolder -> Capacitor_SMD:C_0805_2012Metric_Pad1.18x1.45mm_HandSolder
- C4: renamed from C9; footprint Capacitor_SMD:C_0603_1608Metric -> Capacitor_SMD:C_0805_2012Metric_Pad1.18x1.45mm_HandSolder
- C5: renamed from C1; value 10uF ? -> 10uF; footprint Capacitor_SMD:C_0603_1608Metric -> Capacitor_SMD:C_0805_2012Metric_Pad1.18x1.45mm_HandSolder
- C6: renamed from C7; value C -> 100n; footprint Capacitor_SMD:C_0201_0603Metric_Pad0.64x0.40mm_HandSolder -> Capacitor_SMD:C_0805_2012Metric_Pad1.18x1.45mm_HandSolder
- C7: renamed from C8; value C -> 100n; footprint Capacitor_SMD:C_0201_0603Metric_Pad0.64x0.40mm_HandSolder -> Capacitor_SMD:C_0805_2012Metric_Pad1.18x1.45mm_HandSolder
- R10: renamed from R2; footprint Resistor_SMD:R_0201_0603Metric -> Resistor_SMD:R_0805_2012Metric_Pad1.20x1.40mm_HandSolder
- R11: renamed from R1; footprint Resistor_SMD:R_0201_0603Metric -> Resistor_SMD:R_0805_2012Metric_Pad1.20x1.40mm_HandSolder
- R12: renamed from R9; footprint Resistor_SMD:R_0201_0603Metric -> Resistor_SMD:R_0805_2012Metric_Pad1.20x1.40mm_HandSolder
- R13: renamed from R16; footprint Resistor_SMD:R_0201_0603Metric -> Resistor_SMD:R_0805_2012Metric_Pad1.20x1.40mm_HandSolder
- R14: renamed from R10; footprint Resistor_SMD:R_0201_0603Metric -> Resistor_SMD:R_0805_2012Metric_Pad1.20x1.40mm_HandSolder
- R15: renamed from R17; footprint Resistor_SMD:R_0201_0603Metric -> Resistor_SMD:R_0805_2012Metric_Pad1.20x1.40mm_HandSolder
- R16: renamed from R11; footprint Resistor_SMD:R_0201_0603Metric -> Resistor_SMD:R_0805_2012Metric_Pad1.20x1.40mm_HandSolder
- R17: renamed from R18; footprint Resistor_SMD:R_0201_0603Metric -> Resistor_SMD:R_0805_2012Metric_Pad1.20x1.40mm_HandSolder
- R18: renamed from R4; footprint Resistor_SMD:R_0201_0603Metric -> Resistor_SMD:R_0805_2012Metric_Pad1.20x1.40mm_HandSolder
- R19: renamed from R27; footprint Resistor_SMD:R_0201_0603Metric_Pad0.64x0.40mm_HandSolder -> Resistor_SMD:R_0805_2012Metric_Pad1.20x1.40mm_HandSolder
- R20: renamed from R30; footprint Resistor_SMD:R_0201_0603Metric_Pad0.64x0.40mm_HandSolder -> Resistor_SMD:R_0805_2012Metric_Pad1.20x1.40mm_HandSolder
- R25: renamed from R26; footprint Resistor_SMD:R_0201_0603Metric -> Resistor_SMD:R_0805_2012Metric_Pad1.20x1.40mm_HandSolder
- R3, R8: footprint Resistor_SMD:R_0201_0603Metric -> Resistor_SMD:R_0805_2012Metric_Pad1.20x1.40mm_HandSolder
- R32: renamed from 0-ohm4; value ERJ-2GE0R00X -> 0; footprint ETROC_to_FPGA:RESC1005X40N -> Resistor_SMD:R_0805_2012Metric_Pad1.20x1.40mm_HandSolder
- R33: renamed from 0-ohm5; value ERJ-2GE0R00X -> 0; footprint ETROC_to_FPGA:RESC1005X40N -> Resistor_SMD:R_0805_2012Metric_Pad1.20x1.40mm_HandSolder
- R34: renamed from 0-ohm6; value ERJ-2GE0R00X -> 0; footprint ETROC_to_FPGA:RESC1005X40N -> Resistor_SMD:R_0805_2012Metric_Pad1.20x1.40mm_HandSolder
- R35: renamed from R5; footprint Resistor_SMD:R_0201_0603Metric -> Resistor_SMD:R_0805_2012Metric_Pad1.20x1.40mm_HandSolder
- R36: renamed from R6; footprint Resistor_SMD:R_0201_0603Metric -> Resistor_SMD:R_0805_2012Metric_Pad1.20x1.40mm_HandSolder
- R37: renamed from R31; footprint Resistor_SMD:R_0201_0603Metric_Pad0.64x0.40mm_HandSolder -> Resistor_SMD:R_0805_2012Metric_Pad1.20x1.40mm_HandSolder
- R38: renamed from R32; footprint Resistor_SMD:R_0201_0603Metric_Pad0.64x0.40mm_HandSolder -> Resistor_SMD:R_0805_2012Metric_Pad1.20x1.40mm_HandSolder
- R4: renamed from R12; footprint Resistor_SMD:R_0201_0603Metric -> Resistor_SMD:R_0805_2012Metric_Pad1.20x1.40mm_HandSolder
- R47: renamed from R24; footprint Resistor_SMD:R_0201_0603Metric_Pad0.64x0.40mm_HandSolder -> Resistor_SMD:R_0805_2012Metric_Pad1.20x1.40mm_HandSolder
- R48: renamed from R25; footprint Resistor_SMD:R_0201_0603Metric_Pad0.64x0.40mm_HandSolder -> Resistor_SMD:R_0805_2012Metric_Pad1.20x1.40mm_HandSolder
- R5: renamed from R13; footprint Resistor_SMD:R_0201_0603Metric -> Resistor_SMD:R_0805_2012Metric_Pad1.20x1.40mm_HandSolder
- R55: renamed from 0-ohm3; value ERJ-2GE0R00X -> 0; footprint ETROC_to_FPGA:RESC1005X40N -> Resistor_SMD:R_0805_2012Metric_Pad1.20x1.40mm_HandSolder
- R56: renamed from 0-ohm1; value ERJ-2GE0R00X -> 0; footprint ETROC_to_FPGA:RESC1005X40N -> Resistor_SMD:R_0805_2012Metric_Pad1.20x1.40mm_HandSolder
- R57: renamed from 0-ohm2; value ERJ-2GE0R00X -> 0; footprint ETROC_to_FPGA:RESC1005X40N -> Resistor_SMD:R_0805_2012Metric_Pad1.20x1.40mm_HandSolder
- R6: renamed from R7; footprint Resistor_SMD:R_0201_0603Metric -> Resistor_SMD:R_0805_2012Metric_Pad1.20x1.40mm_HandSolder
- R62: renamed from R20; footprint Resistor_SMD:R_0201_0603Metric_Pad0.64x0.40mm_HandSolder -> Resistor_SMD:R_0805_2012Metric_Pad1.20x1.40mm_HandSolder
- R63: renamed from R23; footprint Resistor_SMD:R_0201_0603Metric_Pad0.64x0.40mm_HandSolder -> Resistor_SMD:R_0805_2012Metric_Pad1.20x1.40mm_HandSolder
- R64: renamed from R33; footprint Resistor_SMD:R_0201_0603Metric_Pad0.64x0.40mm_HandSolder -> Resistor_SMD:R_0805_2012Metric_Pad1.20x1.40mm_HandSolder
- R65: renamed from R34; footprint Resistor_SMD:R_0201_0603Metric_Pad0.64x0.40mm_HandSolder -> Resistor_SMD:R_0805_2012Metric_Pad1.20x1.40mm_HandSolder
- R68: renamed from 0-ohm7; value ERJ-2GE0R00X -> 0; footprint ETROC_to_FPGA:RESC1005X40N -> Resistor_SMD:R_0805_2012Metric_Pad1.20x1.40mm_HandSolder
- R69: renamed from 0-ohm8; value ERJ-2GE0R00X -> 0; footprint ETROC_to_FPGA:RESC1005X40N -> Resistor_SMD:R_0805_2012Metric_Pad1.20x1.40mm_HandSolder
- R7: renamed from R14; footprint Resistor_SMD:R_0201_0603Metric -> Resistor_SMD:R_0805_2012Metric_Pad1.20x1.40mm_HandSolder
- R70: renamed from 0-ohm9; value ERJ-2GE0R00X -> 0; footprint ETROC_to_FPGA:RESC1005X40N -> Resistor_SMD:R_0805_2012Metric_Pad1.20x1.40mm_HandSolder
- R71: renamed from R35; footprint Resistor_SMD:R_0201_0603Metric_Pad0.64x0.40mm_HandSolder -> Resistor_SMD:R_0805_2012Metric_Pad1.20x1.40mm_HandSolder
- R72: renamed from R36; footprint Resistor_SMD:R_0201_0603Metric_Pad0.64x0.40mm_HandSolder -> Resistor_SMD:R_0805_2012Metric_Pad1.20x1.40mm_HandSolder
- R73: renamed from R37; footprint Resistor_SMD:R_0201_0603Metric_Pad0.64x0.40mm_HandSolder -> Resistor_SMD:R_0805_2012Metric_Pad1.20x1.40mm_HandSolder
- R74: renamed from R38; footprint Resistor_SMD:R_0201_0603Metric_Pad0.64x0.40mm_HandSolder -> Resistor_SMD:R_0805_2012Metric_Pad1.20x1.40mm_HandSolder
- R77: renamed from 0-ohm10; value ERJ-2GE0R00X -> 0; footprint ETROC_to_FPGA:RESC1005X40N -> Resistor_SMD:R_0805_2012Metric_Pad1.20x1.40mm_HandSolder
- R78: renamed from 0-ohm11; value ERJ-2GE0R00X -> 0; footprint ETROC_to_FPGA:RESC1005X40N -> Resistor_SMD:R_0805_2012Metric_Pad1.20x1.40mm_HandSolder
- R79: renamed from 0-ohm12; value ERJ-2GE0R00X -> 0; footprint ETROC_to_FPGA:RESC1005X40N -> Resistor_SMD:R_0805_2012Metric_Pad1.20x1.40mm_HandSolder
- R80: renamed from R39; footprint Resistor_SMD:R_0201_0603Metric_Pad0.64x0.40mm_HandSolder -> Resistor_SMD:R_0805_2012Metric_Pad1.20x1.40mm_HandSolder
- R81: renamed from R40; footprint Resistor_SMD:R_0201_0603Metric_Pad0.64x0.40mm_HandSolder -> Resistor_SMD:R_0805_2012Metric_Pad1.20x1.40mm_HandSolder
- R9: renamed from R15; footprint Resistor_SMD:R_0201_0603Metric -> Resistor_SMD:R_0805_2012Metric_Pad1.20x1.40mm_HandSolder
- U2: renamed from U1; value PCA9306 -> PCA9306DCTR
- U3: renamed from U4; value PCA9306 -> PCA9306DCTR
- moved J5 20.0 mm to (36.0, -73.0)
- moved Spacer 20.0 mm to (66.0, -115.0)
- moved Spacer 20.0 mm to (3.01, -115.0)
- moved R72 18.6 mm to (48.9, -64.5)
- moved R71 18.6 mm to (46.6, -64.5)
- moved R37 18.6 mm to (39.8, -64.5)
- moved R38 18.6 mm to (42.0, -64.5)
- moved R32 18.3 mm to (40.9, -57.0)
- moved R68 18.3 mm to (47.7, -57.0)
- moved C21 18.2 mm to (48.9, -59.5)
- moved C20 18.2 mm to (46.6, -59.5)
- moved C6 17.5 mm to (39.8, -59.5)
- moved C7 17.5 mm to (42.0, -59.5)
- moved J6 17.0 mm to (36.0, -105.0)
- moved JP1 16.4 mm to (5.28, -98.2)
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- renumbered J5 to J1, J6 to J2, J7 to J4, J1 to J5, J2 to J6, J3 to J7, TP4 to TP1, TP1 to TP2, TP2 to TP4, U6 to U1, U3 to U4, U2 to U5
Connections:
- C17 pad 1: /FC_P -> /FC_a_P
- C17 pad 2: /FC_P -> /FC_b_P
- C18 pad 1: /FC_N -> /FC_a_N
- C18 pad 2: /FC_N -> /FC_b_N
- C20 pad 1: /DOL_P -> /DOL_a_P
- C20 pad 2: /DOL_P -> /DOL_b_P
- C21 pad 1: /DOL_N -> /DOL_a_N
- C21 pad 2: /DOL_N -> /DOL_b_N
- C22 pad 1: /DOR_P -> /DOR_a_P
- C22 pad 2: /DOR_P -> /DOR_b_P
- C23 pad 1: /DOR_N -> /DOR_a_N
- C23 pad 2: /DOR_N -> /DOR_b_N
- C6 pad 1: /CLK40_P -> /CLK40_a_P
- C6 pad 2: /CLK40_P -> /CLK40_b_P
- C7 pad 1: /CLK40_N -> /CLK40_a_N
- C7 pad 2: /CLK40_N -> /CLK40_b_N
- J5 pad 18: unconnected-(J1-Pad18) -> /RST_WS
- J5 pad 51: /CLK40_P -> /CLK40_b_P
- J5 pad 53: /CLK40_N -> /CLK40_b_N
- J5 pad 55: /CLK1280_P -> unconnected-(J5-Pad55)
- J5 pad 57: /CLK1280_N -> unconnected-(J5-Pad57)
- J5 pad 59: /FC_P -> /FC_b_P
- J5 pad 61: /FC_N -> /FC_b_N
- J5 pad 63: /DOL_P -> /DOL_b_P
- J5 pad 65: /DOL_N -> /DOL_b_N
- J5 pad 67: /DOR_P -> /DOR_b_P
- J5 pad 69: /DOR_N -> /DOR_b_N
- J6 pad 28: unconnected-(J2-Pad28) -> /RSTn
- J7 pad C22: unconnected-(J3-PadC22) -> /CLK40_a_P
- J7 pad C23: unconnected-(J3-PadC23) -> /CLK40_a_N
- J7 pad C26: unconnected-(J3-PadC26) -> /RSTn
- J7 pad D26: unconnected-(J3-PadD26) -> /RST_WS
- J7 pad H10: /DOL_P -> /DOL_a_P
- J7 pad H11: /DOL_N -> /DOL_a_N
- J7 pad H13: /FC_P -> /FC_a_P
- J7 pad H14: /FC_N -> /FC_a_N
- J7 pad H19: /CLK40_P -> unconnected-(J7-PadH19)
- J7 pad H20: /CLK40_N -> unconnected-(J7-PadH20)
- J7 pad H7: /DOR_P -> /DOR_a_P
- J7 pad H8: /DOR_N -> /DOR_a_N
- R19 pad 1: /0.6V -> Net-(R19-Pad1)
- R20 pad 2: /0.6V -> Net-(R19-Pad1)
- R32 pad 1: /0.6V -> Net-(R19-Pad1)
- R33 pad 1: /CLK40_N -> /CLK40_a_N
- R33 pad 2: /CLK40_N -> /CLK40_b_N
- R34 pad 1: /CLK40_P -> /CLK40_a_P
- R34 pad 2: /CLK40_P -> /CLK40_b_P
- R37 pad 1: /CLK40_P -> /CLK40_b_P
- R38 pad 1: /CLK40_N -> /CLK40_b_N
- R47 pad 1: /0.6V -> Net-(R47-Pad1)
- R48 pad 2: /0.6V -> Net-(R47-Pad1)
- R55 pad 1: /0.6V -> Net-(R47-Pad1)
- R56 pad 1: /FC_N -> /FC_a_N
- R56 pad 2: /FC_N -> /FC_b_N
- R57 pad 1: /FC_P -> /FC_a_P
- R57 pad 2: /FC_P -> /FC_b_P
- R62 pad 1: /FC_P -> /FC_b_P
- R63 pad 1: /FC_N -> /FC_b_N
- R64 pad 1: /0.6V -> Net-(R64-Pad1)
- R65 pad 2: /0.6V -> Net-(R64-Pad1)
- R68 pad 1: /0.6V -> Net-(R64-Pad1)
- R69 pad 1: /DOL_N -> /DOL_a_N
- R69 pad 2: /DOL_N -> /DOL_b_N
- R70 pad 1: /DOL_P -> /DOL_a_P
- R70 pad 2: /DOL_P -> /DOL_b_P
- R71 pad 1: /DOL_P -> /DOL_b_P
- R72 pad 1: /DOL_N -> /DOL_b_N
- R73 pad 1: /0.6V -> Net-(R73-Pad1)
- R74 pad 2: /0.6V -> Net-(R73-Pad1)
- R77 pad 1: /0.6V -> Net-(R73-Pad1)
- R78 pad 1: /DOR_N -> /DOR_a_N
- R78 pad 2: /DOR_N -> /DOR_b_N
- R79 pad 1: /DOR_P -> /DOR_a_P
- R79 pad 2: /DOR_P -> /DOR_b_P
- R80 pad 1: /DOR_P -> /DOR_b_P
- R81 pad 1: /DOR_N -> /DOR_b_N
Routing:
- net /RSTn: track 0.00 -> 130.5 mm, vias 0 -> 3
- net /RST_WS: track 0.00 -> 97.9 mm, vias 0 -> 3
- net /CLK40_a_P: track 0.00 -> 64.3 mm, vias 0 -> 1
- net /CLK40_a_N: track 0.00 -> 63.7 mm, vias 0 -> 1
- net /DOL_a_N: track 0.00 -> 52.9 mm, vias 0 -> 1
- net /DOL_a_P: track 0.00 -> 52.9 mm, vias 0 -> 1
- net /FC_P: track 44.3 -> 0.00 mm, vias 1 -> 0
- net /FC_N: track 44.2 -> 0.00 mm, vias 1 -> 0
- net /DOR_N: track 43.1 -> 0.00 mm, vias 1 -> 0
- net /DOR_P: track 43.0 -> 0.00 mm, vias 1 -> 0
- net /CLK40_N: track 42.6 -> 0.00 mm, vias 1 -> 0
- net /CLK40_P: track 42.5 -> 0.00 mm, vias 1 -> 0
- net /DOR_b_P: track 0.00 -> 42.3 mm
- net GND: track 253.3 -> 295.6 mm, vias 166 -> 153
- net /DOR_b_N: track 0.00 -> 42.3 mm
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Other:
- board size 100 x 100 mm -> 100 x 120 mm
- board text added: "ETROC to FPGA v1"
- board text added: "Korea University DREAM LAB"
- board text added: "Power Source XOR 1-2 : EXternal DC3V 2-3 : FPGA_3P3V"
- board text added: "Sungbeom Cho"
- board text added: "VP"
- board text removed: "0.6V"
- board text removed: "0R"
- board text removed: "1-2 : DC3V 2-3 : FPGA_3P3V"
- board text removed: "DO NOT CONNECT BOTH"
- board text removed: "DREAM LAB ETROC to FPGA v1"
- board text removed: "Jumper is available. Since normally LGAD current < 1mA"
- board text removed: "LED_PWR_SRC"
- board text removed: "TP_1.0V"
- board text removed: "TP_1.2V"
- board text removed: "TP_GND"
- board text removed: "TP_PWR_SRC"
- board text removed: "[Warning] Upto 50V!"
