File: ETROC_to_FPGA.kicad_sch (KiCad schematic)
At the start: 83 parts, among them J1 TF06L-80S-0.5SH_800_, J2 TF06L-80S-0.5SH_800_, J3 ASP-134604-01, J4 Conn_01x03_Socket, J5 Conn_Coaxial, J6 Barrel_Jack, J7 Conn_01x03, Q2 NMOS, U1 PCA9306, U2 MIC69502WR, U3 504102B00000G, U4 PCA9306, U6 MIC69502WR

Commit message: Fabricated ETROC_to_FPGA_v1
Parts:
- added 0-ohm1, 0-ohm10, 0-ohm11, 0-ohm12, 0-ohm2, 0-ohm3, 0-ohm4, 0-ohm5, 0-ohm6, 0-ohm7, 0-ohm8, 0-ohm9: ERJ-2GE0R00X, Resistor_SMD:R_0805_2012Metric_Pad1.20x1.40mm_HandSolder, symbol ERJ-2GE0R00X:ERJ-2GE0R00X
- added C10, C11, C13, C14, C15, C16, C8, C9: 100n, Capacitor_SMD:C_0603_1608Metric_Pad1.08x0.95mm_HandSolder, symbol Device:C
- added C19: 10n, Capacitor_SMD:C_0805_2012Metric_Pad1.18x1.45mm_HandSolder, symbol Device:C
- added R21, R22, R23, R24, R43, R44, R45: 1k, Resistor_SMD:R_0603_1608Metric_Pad0.98x0.95mm_HandSolder, symbol Device:R
- added R26, R27, R53, R54, R66, R67, R75, R76: 2.2k, Resistor_SMD:R_0805_2012Metric_Pad1.20x1.40mm_HandSolder, symbol Device:R
- added R28, R29, R30, R31, R49, R50: R, symbol Device:R
- added R39, R40, R41, R42, R58, R59, R60, R61: 50R, Resistor_SMD:R_0805_2012Metric_Pad1.20x1.40mm_HandSolder, symbol Device:R
- added R46: 0-ohm, Resistor_SMD:R_0603_1608Metric_Pad0.98x0.95mm_HandSolder, symbol Device:R
- added R51, R52: 2.2k, symbol Device:R
- C1: renamed from C10; value 10uF ? -> 10uF; footprint Capacitor_SMD:C_0603_1608Metric -> Capacitor_SMD:C_0805_2012Metric_Pad1.18x1.45mm_HandSolder; symbol Device:C_Polarized_Small_US -> Device:C
- C12: renamed from C2; footprint Capacitor_SMD:C_0603_1608Metric -> Capacitor_SMD:C_0805_2012Metric_Pad1.18x1.45mm_HandSolder; symbol Device:C_Polarized_Small_US -> Device:C
- C17: renamed from C5; value C -> 100n; footprint Capacitor_SMD:C_0201_0603Metric_Pad0.64x0.40mm_HandSolder -> Capacitor_SMD:C_0805_2012Metric_Pad1.18x1.45mm_HandSolder; now not fitted
- C18: renamed from C6; value C -> 100n; footprint Capacitor_SMD:C_0201_0603Metric_Pad0.64x0.40mm_HandSolder -> Capacitor_SMD:C_0805_2012Metric_Pad1.18x1.45mm_HandSolder; now not fitted
- C2: renamed from C3; footprint Capacitor_SMD:C_0201_0603Metric_Pad0.64x0.40mm_HandSolder -> Capacitor_SMD:C_0805_2012Metric_Pad1.18x1.45mm_HandSolder
- C20: renamed from C11; value C -> 100n; footprint Capacitor_SMD:C_0201_0603Metric_Pad0.64x0.40mm_HandSolder -> Capacitor_SMD:C_0805_2012Metric_Pad1.18x1.45mm_HandSolder; now not fitted
- C21: renamed from C12; value C -> 100n; footprint Capacitor_SMD:C_0201_0603Metric_Pad0.64x0.40mm_HandSolder -> Capacitor_SMD:C_0805_2012Metric_Pad1.18x1.45mm_HandSolder; now not fitted
- C22: renamed from C13; value C -> 100n; footprint Capacitor_SMD:C_0201_0603Metric_Pad0.64x0.40mm_HandSolder -> Capacitor_SMD:C_0805_2012Metric_Pad1.18x1.45mm_HandSolder; now not fitted
- C23: renamed from C14; value C -> 100n; footprint Capacitor_SMD:C_0201_0603Metric_Pad0.64x0.40mm_HandSolder -> Capacitor_SMD:C_0805_2012Metric_Pad1.18x1.45mm_HandSolder; now not fitted
- C3: renamed from C4; footprint Capacitor_SMD:C_0201_0603Metric_Pad0.64x0.40mm_HandSolder -> Capacitor_SMD:C_0805_2012Metric_Pad1.18x1.45mm_HandSolder
- C4: renamed from C9; footprint Capacitor_SMD:C_0603_1608Metric -> Capacitor_SMD:C_0805_2012Metric_Pad1.18x1.45mm_HandSolder; symbol Device:C_Polarized_Small_US -> Device:C
- C5: renamed from C1; value 10uF ? -> 10uF; footprint Capacitor_SMD:C_0603_1608Metric -> Capacitor_SMD:C_0805_2012Metric_Pad1.18x1.45mm_HandSolder; symbol Device:C_Polarized_Small_US -> Device:C
- C6: renamed from C7; value C -> 100n; footprint Capacitor_SMD:C_0201_0603Metric_Pad0.64x0.40mm_HandSolder -> Capacitor_SMD:C_0805_2012Metric_Pad1.18x1.45mm_HandSolder; now not fitted
- C7: renamed from C8; value C -> 100n; footprint Capacitor_SMD:C_0201_0603Metric_Pad0.64x0.40mm_HandSolder -> Capacitor_SMD:C_0805_2012Metric_Pad1.18x1.45mm_HandSolder; now not fitted
- R10: renamed from R2; footprint Resistor_SMD:R_0201_0603Metric -> Resistor_SMD:R_0805_2012Metric_Pad1.20x1.40mm_HandSolder
- R11: renamed from R1; footprint Resistor_SMD:R_0201_0603Metric -> Resistor_SMD:R_0805_2012Metric_Pad1.20x1.40mm_HandSolder
- R12: renamed from R9; footprint Resistor_SMD:R_0201_0603Metric -> Resistor_SMD:R_0805_2012Metric_Pad1.20x1.40mm_HandSolder
- R13: renamed from R16; footprint Resistor_SMD:R_0201_0603Metric -> Resistor_SMD:R_0805_2012Metric_Pad1.20x1.40mm_HandSolder
- R14: renamed from R10; footprint Resistor_SMD:R_0201_0603Metric -> Resistor_SMD:R_0805_2012Metric_Pad1.20x1.40mm_HandSolder
- R15: renamed from R17; footprint Resistor_SMD:R_0201_0603Metric -> Resistor_SMD:R_0805_2012Metric_Pad1.20x1.40mm_HandSolder
- R16: renamed from R11; footprint Resistor_SMD:R_0201_0603Metric -> Resistor_SMD:R_0805_2012Metric_Pad1.20x1.40mm_HandSolder
- R17: renamed from R18; footprint Resistor_SMD:R_0201_0603Metric -> Resistor_SMD:R_0805_2012Metric_Pad1.20x1.40mm_HandSolder
- R18: renamed from R4; footprint Resistor_SMD:R_0201_0603Metric -> Resistor_SMD:R_0805_2012Metric_Pad1.20x1.40mm_HandSolder
- R19: renamed from R27; footprint Resistor_SMD:R_0201_0603Metric_Pad0.64x0.40mm_HandSolder -> Resistor_SMD:R_0805_2012Metric_Pad1.20x1.40mm_HandSolder
- R20: renamed from R30; footprint Resistor_SMD:R_0201_0603Metric_Pad0.64x0.40mm_HandSolder -> Resistor_SMD:R_0805_2012Metric_Pad1.20x1.40mm_HandSolder
- R25: renamed from R26; footprint Resistor_SMD:R_0201_0603Metric -> Resistor_SMD:R_0805_2012Metric_Pad1.20x1.40mm_HandSolder; Price (none) -> 152KRW
- R3, R8: footprint Resistor_SMD:R_0201_0603Metric -> Resistor_SMD:R_0805_2012Metric_Pad1.20x1.40mm_HandSolder
- R32: renamed from 0-ohm4; value ERJ-2GE0R00X -> 0; footprint RESC1005X40N -> Resistor_SMD:R_0805_2012Metric_Pad1.20x1.40mm_HandSolder; now not fitted
- R33: renamed from 0-ohm5; value ERJ-2GE0R00X -> 0; footprint RESC1005X40N -> Resistor_SMD:R_0805_2012Metric_Pad1.20x1.40mm_HandSolder
- R34: renamed from 0-ohm6; value ERJ-2GE0R00X -> 0; footprint RESC1005X40N -> Resistor_SMD:R_0805_2012Metric_Pad1.20x1.40mm_HandSolder
- R35: renamed from R5; footprint Resistor_SMD:R_0201_0603Metric -> Resistor_SMD:R_0805_2012Metric_Pad1.20x1.40mm_HandSolder
- R36: renamed from R6; footprint Resistor_SMD:R_0201_0603Metric -> Resistor_SMD:R_0805_2012Metric_Pad1.20x1.40mm_HandSolder
- R37: renamed from R31; footprint Resistor_SMD:R_0201_0603Metric_Pad0.64x0.40mm_HandSolder -> Resistor_SMD:R_0805_2012Metric_Pad1.20x1.40mm_HandSolder; now not fitted
- R38: renamed from R32; footprint Resistor_SMD:R_0201_0603Metric_Pad0.64x0.40mm_HandSolder -> Resistor_SMD:R_0805_2012Metric_Pad1.20x1.40mm_HandSolder; now not fitted
- R4: renamed from R12; footprint Resistor_SMD:R_0201_0603Metric -> Resistor_SMD:R_0805_2012Metric_Pad1.20x1.40mm_HandSolder
- R47: renamed from R24; footprint Resistor_SMD:R_0201_0603Metric_Pad0.64x0.40mm_HandSolder -> Resistor_SMD:R_0805_2012Metric_Pad1.20x1.40mm_HandSolder
- R48: renamed from R25; footprint Resistor_SMD:R_0201_0603Metric_Pad0.64x0.40mm_HandSolder -> Resistor_SMD:R_0805_2012Metric_Pad1.20x1.40mm_HandSolder
- R5: renamed from R13; footprint Resistor_SMD:R_0201_0603Metric -> Resistor_SMD:R_0805_2012Metric_Pad1.20x1.40mm_HandSolder
- R55: renamed from 0-ohm3; value ERJ-2GE0R00X -> 0; footprint RESC1005X40N -> Resistor_SMD:R_0805_2012Metric_Pad1.20x1.40mm_HandSolder; now not fitted
- R56: renamed from 0-ohm1; value ERJ-2GE0R00X -> 0; footprint RESC1005X40N -> Resistor_SMD:R_0805_2012Metric_Pad1.20x1.40mm_HandSolder
- R57: renamed from 0-ohm2; value ERJ-2GE0R00X -> 0; footprint RESC1005X40N -> Resistor_SMD:R_0805_2012Metric_Pad1.20x1.40mm_HandSolder
- R6: renamed from R7; footprint Resistor_SMD:R_0201_0603Metric -> Resistor_SMD:R_0805_2012Metric_Pad1.20x1.40mm_HandSolder
- R62: renamed from R20; footprint Resistor_SMD:R_0201_0603Metric_Pad0.64x0.40mm_HandSolder -> Resistor_SMD:R_0805_2012Metric_Pad1.20x1.40mm_HandSolder; now not fitted
- R63: renamed from R23; footprint Resistor_SMD:R_0201_0603Metric_Pad0.64x0.40mm_HandSolder -> Resistor_SMD:R_0805_2012Metric_Pad1.20x1.40mm_HandSolder; now not fitted
- R64: renamed from R33; footprint Resistor_SMD:R_0201_0603Metric_Pad0.64x0.40mm_HandSolder -> Resistor_SMD:R_0805_2012Metric_Pad1.20x1.40mm_HandSolder; now not fitted
- R65: renamed from R34; footprint Resistor_SMD:R_0201_0603Metric_Pad0.64x0.40mm_HandSolder -> Resistor_SMD:R_0805_2012Metric_Pad1.20x1.40mm_HandSolder; now not fitted
- R68: renamed from 0-ohm7; value ERJ-2GE0R00X -> 0; footprint RESC1005X40N -> Resistor_SMD:R_0805_2012Metric_Pad1.20x1.40mm_HandSolder; now not fitted
- R69: renamed from 0-ohm8; value ERJ-2GE0R00X -> 0; footprint RESC1005X40N -> Resistor_SMD:R_0805_2012Metric_Pad1.20x1.40mm_HandSolder
- R7: renamed from R14; footprint Resistor_SMD:R_0201_0603Metric -> Resistor_SMD:R_0805_2012Metric_Pad1.20x1.40mm_HandSolder
- R70: renamed from 0-ohm9; value ERJ-2GE0R00X -> 0; footprint RESC1005X40N -> Resistor_SMD:R_0805_2012Metric_Pad1.20x1.40mm_HandSolder
- R71: renamed from R35; footprint Resistor_SMD:R_0201_0603Metric_Pad0.64x0.40mm_HandSolder -> Resistor_SMD:R_0805_2012Metric_Pad1.20x1.40mm_HandSolder; now not fitted
- R72: renamed from R36; footprint Resistor_SMD:R_0201_0603Metric_Pad0.64x0.40mm_HandSolder -> Resistor_SMD:R_0805_2012Metric_Pad1.20x1.40mm_HandSolder; now not fitted
- R73: renamed from R37; footprint Resistor_SMD:R_0201_0603Metric_Pad0.64x0.40mm_HandSolder -> Resistor_SMD:R_0805_2012Metric_Pad1.20x1.40mm_HandSolder
- R74: renamed from R38; footprint Resistor_SMD:R_0201_0603Metric_Pad0.64x0.40mm_HandSolder -> Resistor_SMD:R_0805_2012Metric_Pad1.20x1.40mm_HandSolder
- R77: renamed from 0-ohm10; value ERJ-2GE0R00X -> 0; footprint RESC1005X40N -> Resistor_SMD:R_0805_2012Metric_Pad1.20x1.40mm_HandSolder; now not fitted
- R78: renamed from 0-ohm11; value ERJ-2GE0R00X -> 0; footprint RESC1005X40N -> Resistor_SMD:R_0805_2012Metric_Pad1.20x1.40mm_HandSolder
- R79: renamed from 0-ohm12; value ERJ-2GE0R00X -> 0; footprint RESC1005X40N -> Resistor_SMD:R_0805_2012Metric_Pad1.20x1.40mm_HandSolder
- R80: renamed from R39; footprint Resistor_SMD:R_0201_0603Metric_Pad0.64x0.40mm_HandSolder -> Resistor_SMD:R_0805_2012Metric_Pad1.20x1.40mm_HandSolder; now not fitted
- R81: renamed from R40; footprint Resistor_SMD:R_0201_0603Metric_Pad0.64x0.40mm_HandSolder -> Resistor_SMD:R_0805_2012Metric_Pad1.20x1.40mm_HandSolder; now not fitted
- R9: renamed from R15; footprint Resistor_SMD:R_0201_0603Metric -> Resistor_SMD:R_0805_2012Metric_Pad1.20x1.40mm_HandSolder
- U2: renamed from U1; value PCA9306 -> PCA9306DCTR
- U3: renamed from U4; value PCA9306 -> PCA9306DCTR
- renumbered D2 to D1, J5 to J1, J6 to J2, J4 to J3, J7 to J4, J1 to J5, J2 to J6, J3 to J7, Q2 to Q1, R28 to R1, R29 to R2, TP4 to TP1, TP1 to TP2, TP2 to TP4, U6 to U1, U3 to U4, U2 to U5
Connections:
- net 0.6V: now also 0-ohm1.1, 0-ohm4.1, 0-ohm7.1, R21.1, R22.2, R23.1, R24.2, R28.2, R29.1, R30.2, R31.1, R43.1, R44.2, R49.2, R50.1; no longer R19.1, R20.2, R32.1, R47.1, R48.2, R55.1, R64.1, R65.2, R68.1, R73.1, R74.2, R77.1
- net 1.2V: now also 0-ohm9.1, R21.2, R23.2, R43.2, R45.1, R45.2, R46.2, R51.2, R52.1
- net CLK1280_N: no longer J5.57
- net CLK1280_P: no longer J5.55
- net GND: now also C19.1, R22.1, R24.1, R44.1, R46.1
- net VP: now also C19.2
- net RST_WS: now reaches J5.18
- net RST_WS: now also J7.D26
- net RSTn: now reaches J6.28
- net RSTn: now also J7.C26
- net CLK40_a_P: now reaches J7.C22
- net CLK40_a_P: now also C6.1, R34.1, R26.1
- net CLK40_a_N: now reaches J7.C23
- net CLK40_a_N: now also C7.1, R33.1, R27.1
- net CLK40_N renamed CLK40_b_N
- net CLK40_b_N: no longer C7.1, J7.H20, R33.1
- net CLK40_P renamed CLK40_b_P
- net CLK40_b_P: no longer C6.1, J7.H19, R34.1
- net DOL_N renamed DOL_b_N
- net DOL_b_N: no longer C21.1, J7.H11, R69.1
- net DOL_P renamed DOL_b_P
- net DOL_b_P: no longer C20.1, J7.H10, R70.1
- net DOR_N renamed DOR_b_N
- net DOR_b_N: no longer C23.1, J7.H8, R78.1
- net DOR_P renamed DOR_b_P
- net DOR_b_P: no longer C22.1, J7.H7, R79.1
- net FC_N renamed FC_b_N
- net FC_b_N: no longer C18.1, J7.H14, R56.1
- net FC_P renamed FC_b_P
- net FC_b_P: no longer C17.1, J7.H13, R57.1
- new net: R47.1, R48.2, R53.2, R54.2, R55.1
- new net: R64.1, R65.2, R66.2, R67.2, R68.1
- new net: R73.1, R74.2, R75.2, R76.2, R77.1
- new net: 0-ohm1.2, R39.2, R40.2
- new net: 0-ohm4.2, R41.2, R42.2
- new net: 0-ohm9.2, R60.2, R61.2
- new net: R19.1, R20.2, R26.2, R27.2, R32.1
- new net: 0-ohm7.2, R58.2, R59.2
- new net DOL_a_N: C21.1, J7.H11, R67.1, R69.1
- new net DOL_a_P: C20.1, J7.H10, R66.1, R70.1
- new net DOR_a_N: C23.1, J7.H8, R76.1, R78.1
- new net DOR_a_P: C22.1, J7.H7, R75.1, R79.1
- new net Diff_N: 0-ohm10.1, 0-ohm10.2, 0-ohm2.1, 0-ohm2.2, 0-ohm5.1, 0-ohm5.2, 0-ohm8.1, 0-ohm8.2, C11.1, C11.2, C14.1, C14.2, C16.1, C16.2, C9.1, C9.2, R29.2, R31.2, R40.1, R42.1, R50.2, R52.2, R59.1, R61.1
- new net Diff_P: 0-ohm11.1, 0-ohm11.2, 0-ohm12.1, 0-ohm12.2, 0-ohm3.1, 0-ohm3.2, 0-ohm6.1, 0-ohm6.2, C10.1, C10.2, C13.1, C13.2, C15.1, C15.2, C8.1, C8.2, R28.1, R30.1, R39.1, R41.1, R49.1, R51.1, R58.1, R60.1
- new net FC_a_N: C18.1, J7.H14, R54.1, R56.1
- new net FC_a_P: C17.1, J7.H13, R53.1, R57.1
- no-connect marks 9 -> 92
Other:
- note added: "(Optional) Sinking path for Leakage Current from PCA9306 to LDO"
- note added: "*or 2.2k"
- note added: "0-ohm"
- note added: "1"
- note added: "10uF"
- note added: "2"
- note added: "DNP"
- note added: "DP_0402"
- note added: "Example"
- note added: "If use ETROC internal termination, populate 2.2kR"
- note added: "LVDS (1.2V) to CLPS (0.6V) If Forward Board (Original) : 1. DNP Capacitor-bypassing 0-ohms. 2. Populate 0.6V 0-ohm. If use ETROC internal termination : 1. Populate 2.2kR resistors instead of 50R. If Reverse Board, 1. Bypass Capacitor using 0ohm. 2. DNP terminal 50+50R 3. DNP 0.6V 0-ohm"
- note added: "Receiving CLPS"
- note added: "Receiving LVDS"
- note added: "Sending CLPS"
- note added: "Sending LVDS"
- note removed: "LVDS (1.2V) to CLPS (0.6V) If Reverse Board, 1. Bypass Capacitor using 0ohm. 2. DNP terminal 50+50R"
- moved on the sheet: C2, C3, D1, Q1, R1, R12, R13, R14, R15, R16, R17, R19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

Commit message: Fabricated ETROC_to_FPGA_v1
Other:
- note added: "Board Design : Sungbeom Cho (sucho@cern.ch)"
- note added: "ETROC_to_FPGA_v1"
- note added: "Institution : Korea University DREAM Group"
- moved on the sheet: C1, C12, C19, C2, C3, C4, C5, D1, J1, J2, J3, J4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
